File: kicad/sensor-umidade/sensor-umidade.kicad_pcb (KiCad board)
At the start: 2 copper layers, 4 parts, among them Q1 BC549

Commit message: kicad sensor PCB done
Parts:
- added J1: Conn_01x01_MountingPin, Connector_Pin:Pin_D1.0mm_L10.0mm, F.Cu at (113.0, -54.6)
- added J2: Conn_01x01_MountingPin, Connector_Pin:Pin_D1.0mm_L10.0mm, F.Cu at (113.0, -49.5)
- added J3: Conn_01x01_MountingPin, Connector_Pin:Pin_D1.0mm_L10.0mm, F.Cu at (82.5, -45.7)
- added J4: Conn_01x01_MountingPin, Connector_Pin:Pin_D1.0mm_L10.0mm, F.Cu at (82.5, -55.9)
Routing:
- net +3V0: track 0.00 -> 34.3 mm
- net Net-(J1-Pad1): track 0.00 -> 7.63 mm
- net GND: track 0.00 -> 7.62 mm
- net Net-(Q1-Pad2): track 0.00 -> 5.09 mm
- net Net-(Q1-Pad1): track 0.00 -> 3.81 mm
- net Net-(D1-Pad1): track 0.00 -> 3.81 mm
Other:
- board text added: "robotizando.com.br/pt-br/agua-na-planta"
